File: CE6A.brd (EAGLE design)
At the start: 55 x 37 mm, 43 parts, among them IC1 LM358, Q1 40N03, T1 BC847, U1 TL431ASA-7

Commit message: Update
Parts:
- added U$3, U$4: (no value), xdesig:OSHW_ES000052
Changed lines of the file:
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@@
 <grid distance="0.05" unitdist="inch" unit="mm" style="lines" multiple="1" display="no" altdistance="0.15875" altunitdist="mm" altunit="mm"/>
 <layers>
-<layer number="1" name="Top" color="1" fill="1" visible="yes" active="yes"/>
+<layer number="1" name="Top" color="1" fill="1" visible="no" active="yes"/>
 <layer number="2" name="Route2" color="1" fill="3" visible="no" active="no"/>
 <layer number="3" name="Route3" color="4" fill="3" visible="no" active="no"/>
@@
 <layer number="19" name="Unrouted" color="6" fill="1" visible="yes" active="yes"/>
 <layer number="20" name="Dimension" color="15" fill="1" visible="yes" active="yes"/>
-<layer number="21" name="tPlace" color="7" fill="1" visible="yes" active="yes"/>
-<layer number="22" name="bPlace" color="7" fill="1" visible="no" active="yes"/>
+<layer number="21" name="tPlace" color="7" fill="1" visible="no" active="yes"/>
+<layer number="22" name="bPlace" color="7" fill="1" visible="yes" active="yes"/>
 <layer number="23" name="tOrigins" color="15" fill="1" visible="no" active="yes"/>
-<layer number="24" name="bOrigins" color="15" fill="1" visible="no" active="yes"/>
+<layer number="24" name="bOrigins" color="15" fill="1" visible="yes" active="yes"/>
 <layer number="25" name="tNames" color="7" fill="1" visible="no" active="yes"/>
-<layer number="26" name="bNames" color="7" fill="1" visible="no" active="yes"/>
+<layer number="26" name="bNames" color="7" fill="1" visible="yes" active="yes"/>
 <layer number="27" name="tValues" color="7" fill="1" visible="no" active="yes"/>
 <layer number="28" name="bValues" color="7" fill="1" visible="no" active="yes"/>
@@
 <layer number="30" name="bStop" color="7" fill="6" visible="no" active="yes"/>
 <layer number="31" name="tCream" color="7" fill="4" visible="no" active="yes"/>
-<layer number="32" name="bCream" color="7" fill="5" visible="no" active="yes"/>
+<layer number="32" name="bCream" color="7" fill="5" visible="yes" active="yes"/>
 <layer number="33" name="tFinish" color="6" fill="3" visible="no" active="yes"/>
 <layer number="34" name="bFinish" color="6" fill="6" visible="no" active="yes"/>
@@
 x + -
 </text>
-<text x="20.79625" y="5.715" size="1.27" layer="21" font="vector" rot="R180">VAdj</text>
+<text x="16.03375" y="5.08" size="1.27" layer="21" font="vector" rot="R270">VAdj</text>
 <text x="12.99" y="18.5" size="1.016" layer="16" font="vector" ratio="10" rot="MR90" align="center">Deseñado en Estrimia con Agarimo
 CERN-OHL-S-2.0</text>
@@
 <text x="30.63875" y="30.1625" size="1.27" layer="21" font="vector" align="center">GND</text>
 <text x="49.05375" y="25.0825" size="2.54" layer="21" font="vector" rot="R270" align="center">GDS</text>
-<text x="4.92125" y="21.11375" size="1.778" layer="21" font="vector" align="center">12Vcc</text>
+<text x="4.92125" y="20.47875" size="1.778" layer="21" font="vector" align="center">12Vcc</text>
 <text x="34.44875" y="3.96875" size="1.778" layer="21" font="vector" rot="R90" align="center">Corr</text>
 <text x="23.1775" y="30.1625" size="1.27" layer="21" font="vector" align="center">12Vcc</text>
@@
 <text x="3.81" y="18.5" size="1.27" layer="16" font="vector" rot="MR270" align="center">EL6A V001
 2415</text>
-<text x="33.49625" y="18.5" size="1.27" layer="16" font="vector" rot="MR270" align="center">XDeSIG</text>
-<text x="14.12875" y="33.02" size="2.1844" layer="21" font="vector" align="center">CE6A</text>
+<text x="29.21" y="18.34125" size="1.27" layer="16" font="vector" rot="MR270" align="center">XDeSIG</text>
+<text x="17.145" y="7.14375" size="2.1844" layer="21" font="vector" rot="R180" align="center">CE6A</text>
 <text x="27.46375" y="5.3975" size="0.8128" layer="21" font="vector" align="center">RV09
 10K</text>
@@
 <attribute name="MF" value="" x="52.3875" y="13.97" size="1.778" layer="27" rot="R270" display="off"/>
 <attribute name="OC_FARNELL" value="unknown" x="52.3875" y="13.97" size="1.778" layer="27" rot="R270" display="off"/>
-<attribute name="NAME" x="48.5775" y="7.366" size="0.8128" layer="25" font="vector" ratio="10"/>
 <attribute name="VALUE" x="54.0385" y="13.97" size="1.27" layer="27" ratio="10" rot="R270"/>
 </element>
@@
 <attribute name="VALUE" x="53.6575" y="24.92375" size="0.0254" layer="28" rot="MR180"/>
 </element>
+<element name="U$3" library="xdesig" package="OSHW_ES000052" value="" x="8.89" y="30.32125"/>
+<element name="U$4" library="xdesig" package="OSHW_ES000052" value="" x="20.47875" y="14.76375" rot="MR90"/>
 </elements>
 <signals>
